Commit message: converted description to xacro macro, added standalone version

File: urdf/sting_carriage.xacro (robot description, xacro)
@@ -1,231 +1,231 @@
 <robot
-    name="sting_carriage"
     xmlns:xacro="http://www.ros.org/wiki/xacro">
-    <link name="carriage_base_link" />
-    <link
-        name="carriage_base">
-        <inertial>
-            <origin
-                xyz="0.167060618559883 3.79365166004036E-06 -0.00965640428281041"
-                rpy="0 0 0" />
-            <mass
-                value="0.699726153260739" />
-            <inertia
-                ixx="0.000529149363493783"
-                ixy="4.66130830711204E-07"
-                ixz="0.000555748330443739"
-                iyy="0.0294300280099401"
-                iyz="-2.93910039380959E-08"
-                izz="0.0296524811775225" />
-        </inertial>
-        <visual>
+    <xacro:macro name="sting_carriage" params="base_link payload:=payload">
+        <link
+            name="carriage_base">
+            <inertial>
+                <origin
+                    xyz="0.167060618559883 3.79365166004036E-06 -0.00965640428281041"
+                    rpy="0 0 0" />
+                <mass
+                    value="0.699726153260739" />
+                <inertia
+                    ixx="0.000529149363493783"
+                    ixy="4.66130830711204E-07"
+                    ixz="0.000555748330443739"
+                    iyy="0.0294300280099401"
+                    iyz="-2.93910039380959E-08"
+                    izz="0.0296524811775225" />
+            </inertial>
+            <visual>
+                <origin
+                    xyz="0 0 0"
+                    rpy="0 0 0" />
+                <geometry>
+                    <mesh
+                        filename="package://sting_carriage_description/meshes/carriage_base.STL" />
+                </geometry>
+                <material
+                    name="">
+                    <color
+                        rgba="1 1 1 1" />
+                </material>
+            </visual>
+            <collision>
+                <origin
+                    xyz="0 0 0"
+                    rpy="0 0 0" />
+                <geometry>
+                    <mesh
+                        filename="package://sting_carriage_description/meshes/carriage_base_collision.STL" />
+                </geometry>
+            </collision>
+        </link>
+        <joint name="sting_carriage_base_joint"
+            type="fixed">
             <origin
                 xyz="0 0 0"
                 rpy="0 0 0" />
-            <geometry>
-                <mesh
-                    filename="package://sting_carriage_description/meshes/carriage_base.STL" />
-            </geometry>
-            <material
-                name="">
-                <color
-                    rgba="1 1 1 1" />
-            </material>
-        </visual>
-        <collision>
-            <origin
-                xyz="0 0 0"
-                rpy="0 0 0" />
-            <geometry>
-                <mesh
-                    filename="package://sting_carriage_description/meshes/carriage_base_collision.STL" />
-            </geometry>
-        </collision>
-    </link>
-    <joint name="base_joint"
-        type="fixed">
-        <origin
-            xyz="0 0 0"
-            rpy="0 0 0" />
-        <parent
-            link="carriage_base_link" />
-        <child
-            link="carriage_base" />
-    </joint>
-    <link
-        name="carriage_slider">
-        <inertial>
-            <origin
-                xyz="0.000156693213846357 -0.0618128630425778 -0.00323427667463473"
-                rpy="0 0 0" />
-            <mass
-                value="0.112932852597131" />
-            <inertia
-                ixx="0.000168948390924987"
-                ixy="1.2159591448882E-08"
-                ixz="-8.88631626187684E-08"
-                iyy="0.000168996514994476"
-                iyz="6.3343116038627E-07"
-                izz="0.000329383199257969" />
-        </inertial>
-        <visual>
-            <origin
-                xyz="0 0 0"
-                rpy="0 0 0" />
-            <geometry>
-                <mesh
-                    filename="package://sting_carriage_description/meshes/carriage_slider.STL" />
-            </geometry>
-            <material
-                name="">
-                <color
-                    rgba="0.792156862745098 0.819607843137255 0.933333333333333 1" />
-            </material>
-        </visual>
-        <collision>
-            <origin
-                xyz="0 0 0"
-                rpy="0 0 0" />
-            <geometry>
-                <mesh
-                    filename="package://sting_carriage_description/meshes/carriage_slider_collision.STL" />
-            </geometry>
-        </collision>
-    </link>
-    <joint
-        name="slider_joint"
-        type="prismatic">
-        <origin
-            xyz="0 0 0.0123"
-            rpy="-2.612E-14 1.2049E-14 1.5708" />
-        <parent
-            link="carriage_base" />
-        <child
-            link="carriage_slider" />
-        <axis
-            xyz="0 -1 0" />
-        <limit
-            lower="0"
-            upper="0.4"
-            effort="1.1"
-            velocity="0.2" />
-    </joint>
-    <link
-        name="payload" />
-    <joint
-        name="payload_joint"
-        type="fixed">
-        <origin
-            xyz="0.0430500000000003 -0.0625000000000459 0.00300000000000002"
-            rpy="3.15544362088405E-30 -7.26931742313452E-18 7.23883640127473E-17" />
-        <parent
-            link="carriage_slider" />
-        <child
-            link="payload" />
-        <axis
-            xyz="0 0 0" />
-    </joint>
-    <link
-        name="sensor_reading_surface" />
-    <joint
-        name="sensor_reading_joint"
-        type="fixed">
-        <origin
-            xyz="0 -0.02 0.0205"
-            rpy="0 -7.26931742313452E-18 1.69981808512144E-16" />
-        <parent
-            link="carriage_slider" />
-        <child
-            link="sensor_reading_surface" />
-        <axis
-            xyz="0 0 0" />
-    </joint>
-    <link
-        name="right_sensor">
-        <inertial>
-            <origin
-                xyz="-0.0017532582061619 4.27804446363547E-05 0.00214459124724793"
-                rpy="0 0 0" />
-            <mass
-                value="0.00031258592156757" />
-            <inertia
-                ixx="1.16655193608404E-08"
-                ixy="1.30303505907792E-11"
-                ixz="2.18898551781116E-11"
-                iyy="2.77078095612999E-09"
-                iyz="-1.73164791414335E-12"
-                izz="9.07515985909764E-09" />
-        </inertial>
-        <visual>
-            <origin
-                xyz="0 0 0"
-                rpy="0 0 0" />
-            <geometry>
-                <mesh
-                    filename="package://sting_carriage_description/meshes/right_sensor.STL" />
-            </geometry>
-            <material
-                name="">
-                <color
-                    rgba="0.6 0.6 0.6 1" />
-            </material>
-        </visual>
-    </link>
-    <joint
-        name="right_sensor_joint"
-        type="fixed">
-        <origin
-            xyz="-0.0422 -0.01498 0.03177"
-            rpy="4.8187E-17 0 0" />
-        <parent
-            link="carriage_base" />
-        <child
-            link="right_sensor" />
-        <axis
-            xyz="0 0 0" />
-    </joint>
-    <link
-        name="left_sensor">
-        <inertial>
-            <origin
-                xyz="-0.0017532582061619 4.27804446363478E-05 0.00214459124724793"
-                rpy="0 0 0" />
-            <mass
-                value="0.000312585921567569" />
-            <inertia
-                ixx="1.16655193608404E-08"
-                ixy="1.30303505907791E-11"
-                ixz="2.18898551781117E-11"
-                iyy="2.77078095612999E-09"
-                iyz="-1.7316479141429E-12"
-                izz="9.07515985909763E-09" />
-        </inertial>
-        <visual>
-            <origin
-                xyz="0 0 0"
-                rpy="0 0 0" />
-            <geometry>
-                <mesh
-                    filename="package://sting_carriage_description/meshes/left_sensor.STL" />
-            </geometry>
-            <material
-                name="">
-                <color
-                    rgba="0.6 0.6 0.6 1" />
-            </material>
-        </visual>
-    </link>
-    <joint
-        name="left_sensor_joint"
-        type="fixed">
-        <origin
-            xyz="-0.0421999999999995 0.0150200728763124 0.0317700000000001"
-            rpy="4.8186763221578E-17 0 0" />
-        <parent
-            link="carriage_base" />
-        <child
-            link="left_sensor" />
-        <axis
-            xyz="0 0 0" />
-    </joint>
+            <parent
+                link="${base_link}" />
+            <child
+                link="carriage_base" />
+        </joint>
+        <link
+            name="carriage_slider">
+            <inertial>
+                <origin
+                    xyz="0.000156693213846357 -0.0618128630425778 -0.00323427667463473"
+                    rpy="0 0 0" />
+                <mass
+                    value="0.112932852597131" />
+                <inertia
+                    ixx="0.000168948390924987"
+                    ixy="1.2159591448882E-08"
+                    ixz="-8.88631626187684E-08"
+                    iyy="0.000168996514994476"
+                    iyz="6.3343116038627E-07"
+                    izz="0.000329383199257969" />
+            </inertial>
+            <visual>
+                <origin
+                    xyz="0 0 0"
+                    rpy="0 0 0" />
+                <geometry>
+                    <mesh
+                        filename="package://sting_carriage_description/meshes/carriage_slider.STL" />
+                </geometry>
+                <material
+                    name="">
+                    <color
+                        rgba="0.792156862745098 0.819607843137255 0.933333333333333 1" />
+                </material>
+            </visual>
+            <collision>
+                <origin
+                    xyz="0 0 0"
+                    rpy="0 0 0" />
+                <geometry>
+                    <mesh
+                        filename="package://sting_carriage_description/meshes/carriage_slider_collision.STL" />
+                </geometry>
+            </collision>
+        </link>
+        <joint
+            name="slider_joint"
+            type="prismatic">
+            <origin
+                xyz="0 0 0.0123"
+                rpy="-2.612E-14 1.2049E-14 1.5708" />
+            <parent
+                link="carriage_base" />
+            <child
+                link="carriage_slider" />
+            <axis
+                xyz="0 -1 0" />
+            <limit
+                lower="0"
+                upper="0.4"
+                effort="1.1"
+                velocity="0.2" />
+        </joint>
+        <link
+            name="${payload}" />
+        <joint
+            name="payload_joint"
+            type="fixed">
+            <origin
+                xyz="0.0430500000000003 -0.0625000000000459 0.00300000000000002"
+                rpy="3.15544362088405E-30 -7.26931742313452E-18 7.23883640127473E-17" />
+            <parent
+                link="carriage_slider" />
+            <child
+                link="${payload}" />
+            <axis
+                xyz="0 0 0" />
+        </joint>
+        <link
+            name="sensor_reading_surface" />
+        <joint
+            name="sensor_reading_joint"
+            type="fixed">
+            <origin
+                xyz="0 -0.02 0.0205"
+                rpy="0 -7.26931742313452E-18 1.69981808512144E-16" />
+            <parent
+                link="carriage_slider" />
+            <child
+                link="sensor_reading_surface" />
+            <axis
+                xyz="0 0 0" />
+        </joint>
+        <link
+            name="right_sensor">
+            <inertial>
+                <origin
+                    xyz="-0.0017532582061619 4.27804446363547E-05 0.00214459124724793"
+                    rpy="0 0 0" />
+                <mass
+                    value="0.00031258592156757" />
+                <inertia
+                    ixx="1.16655193608404E-08"
+                    ixy="1.30303505907792E-11"
+                    ixz="2.18898551781116E-11"
+                    iyy="2.77078095612999E-09"
+                    iyz="-1.73164791414335E-12"
+                    izz="9.07515985909764E-09" />
+            </inertial>
+            <visual>
+                <origin
+                    xyz="0 0 0"
+                    rpy="0 0 0" />
+                <geometry>
+                    <mesh
+                        filename="package://sting_carriage_description/meshes/right_sensor.STL" />
+                </geometry>
+                <material
+                    name="">
+                    <color
+                        rgba="0.6 0.6 0.6 1" />
+                </material>
+            </visual>
+        </link>
+        <joint
+            name="right_sensor_joint"
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
Commit message: updated robot description

File: urdf/sting_carriage.xacro (robot description, xacro)
@@ -2,19 +2,27 @@
     xmlns:xacro="http://www.ros.org/wiki/xacro">
     <xacro:macro name="sting_carriage" params="base_link payload:=payload">
+        <joint
+            name="carriage_base_joint"
+            type="fixed">
+            <parent
+                link="${base_link}" />
+            <child
+                link="carriage_base" />
+        </joint>
         <link
             name="carriage_base">
             <inertial>
                 <origin
-                    xyz="0.167060618559883 3.79365166004036E-06 -0.00965640428281041"
+                    xyz="0.168470001541672 3.81834085849686E-06 -0.00990038826765847"
                     rpy="0 0 0" />
                 <mass
-                    value="0.699726153260739" />
+                    value="0.695201759420563" />
                 <inertia
-                    ixx="0.000529149363493783"
-                    ixy="4.66130830711204E-07"
-                    ixz="0.000555748330443739"
-                    iyy="0.0294300280099401"
-                    iyz="-2.93910039380959E-08"
-                    izz="0.0296524811775225" />
+                    ixx="0.000521513476559902"
+                    ixy="4.69872062195191E-07"
+                    ixz="0.00051877667389809"
+                    iyy="0.0292099358589963"
+                    iyz="-3.00386636426339E-08"
+                    izz="0.0294377821647163" />
             </inertial>
             <visual>
@@ -42,19 +50,9 @@
             </collision>
         </link>
-        <joint name="sting_carriage_base_joint"
-            type="fixed">
-            <origin
-                xyz="0 0 0"
-                rpy="0 0 0" />
-            <parent
-                link="${base_link}" />
-            <child
-                link="carriage_base" />
-        </joint>
         <link
             name="carriage_slider">
             <inertial>
                 <origin
-                    xyz="0.000156693213846357 -0.0618128630425778 -0.00323427667463473"
+                    xyz="0.000156693213846128 -0.0618128630425793 -0.00323427667463495"
                     rpy="0 0 0" />
                 <mass
@@ -62,8 +60,8 @@
                 <inertia
                     ixx="0.000168948390924987"
-                    ixy="1.2159591448882E-08"
-                    ixz="-8.88631626187684E-08"
+                    ixy="1.21595914488396E-08"
+                    ixz="-8.88631626187852E-08"
                     iyy="0.000168996514994476"
-                    iyz="6.3343116038627E-07"
+                    iyz="6.33431160386277E-07"
                     izz="0.000329383199257969" />
             </inertial>
@@ -79,5 +77,5 @@
                     name="">
                     <color
-                        rgba="0.792156862745098 0.819607843137255 0.933333333333333 1" />
+                        rgba="1 1 1 1" />
                 </material>
             </visual>
@@ -96,6 +94,6 @@
             type="prismatic">
             <origin
-                xyz="0 0 0.0123"
-                rpy="-2.612E-14 1.2049E-14 1.5708" />
+                xyz="0.00600000000000045 0 0.0123000000000001"
+                rpy="-2.61195978578554E-14 1.20485688601907E-14 1.57079632679491" />
             <parent
                 link="carriage_base" />
@@ -106,10 +104,9 @@
             <limit
                 lower="0"
-                upper="0.4"
+                upper="0.367"
                 effort="1.1"
                 velocity="0.2" />
         </joint>
-        <link
-            name="${payload}" />
+        <link name="${payload}" />
         <joint
             name="payload_joint"
@@ -125,107 +122,4 @@
                 xyz="0 0 0" />
         </joint>
-        <link
-            name="sensor_reading_surface" />
-        <joint
-            name="sensor_reading_joint"
-            type="fixed">
-            <origin
-                xyz="0 -0.02 0.0205"
-                rpy="0 -7.26931742313452E-18 1.69981808512144E-16" />
-            <parent
-                link="carriage_slider" />
-            <child
-                link="sensor_reading_surface" />
-            <axis
-                xyz="0 0 0" />
-        </joint>
-        <link
-            name="right_sensor">
-            <inertial>
-                <origin
-                    xyz="-0.0017532582061619 4.27804446363547E-05 0.00214459124724793"
-                    rpy="0 0 0" />
-                <mass
-                    value="0.00031258592156757" />
-                <inertia
-                    ixx="1.16655193608404E-08"
-                    ixy="1.30303505907792E-11"
-                    ixz="2.18898551781116E-11"
-                    iyy="2.77078095612999E-09"
-                    iyz="-1.73164791414335E-12"
-                    izz="9.07515985909764E-09" />
-            </inertial>
-            <visual>
-                <origin
-                    xyz="0 0 0"
-                    rpy="0 0 0" />
-                <geometry>
-                    <mesh
-                        filename="package://sting_carriage_description/meshes/right_sensor.STL" />
-                </geometry>
-                <material
-                    name="">
-                    <color
-                        rgba="0.6 0.6 0.6 1" />
-                </material>
-            </visual>
-        </link>
-        <joint
-            name="right_sensor_joint"
-            type="fixed">
-            <origin
-                xyz="-0.0422 -0.01498 0.03177"
-                rpy="4.8187E-17 0 0" />
-            <parent
-                link="carriage_base" />
-            <child
-                link="right_sensor" />
-            <axis
-                xyz="0 0 0" />
-        </joint>
-        <link
-            name="left_sensor">
-            <inertial>
-                <origin
-                    xyz="-0.0017532582061619 4.27804446363478E-05 0.00214459124724793"
-                    rpy="0 0 0" />
-                <mass
-                    value="0.000312585921567569" />
-                <inertia
-                    ixx="1.16655193608404E-08"
-                    ixy="1.30303505907791E-11"
-                    ixz="2.18898551781117E-11"
-                    iyy="2.77078095612999E-09"
-                    iyz="-1.7316479141429E-12"
-                    izz="9.07515985909763E-09" />
-            </inertial>
-            <visual>
-                <origin
-                    xyz="0 0 0"
-                    rpy="0 0 0" />
-                <geometry>
-                    <mesh
-                        filename="package://sting_carriage_description/meshes/left_sensor.STL" />
-                </geometry>
-                <material
-                    name="">
-                    <color
-                        rgba="0.6 0.6 0.6 1" />
-                </material>
-            </visual>
-        </link>
-        <joint
-            name="left_sensor_joint"
-            type="fixed">
-            <origin
-                xyz="-0.0421999999999995 0.0150200728763124 0.0317700000000001"
-                rpy="4.8186763221578E-17 0 0" />
-            <parent
-                link="carriage_base" />
-            <child
-                link="left_sensor" />
-            <axis
-                xyz="0 0 0" />
-        </joint>
     </xacro:macro>
 </robot>
